Commit message: feat(driver): change ctrl_param_duration_ms to 55

File: brainco_hardware/stark_ethercat/brainco_hand_ethercat_driver/config/revo2_left.ros2_control.xacro (robot description, xacro)
@@ -1,5 +1,5 @@
 <?xml version="1.0"?>
 <robot xmlns:xacro="http://www.ros.org/wiki/xacro">
-    <xacro:macro name="revo2_left_ros2_control" params="name initial_positions_file ctrl_param_duration_ms:=10">
+    <xacro:macro name="revo2_left_ros2_control" params="name initial_positions_file ctrl_param_duration_ms:=55">
         <xacro:property name="initial_positions" value="${xacro.load_yaml(initial_positions_file)['initial_positions']}"/>
         <ros2_control name="${name}" type="system">

File: brainco_hardware/stark_ethercat/brainco_hand_ethercat_driver/config/revo2_left.urdf.xacro (robot description, xacro)
@@ -2,5 +2,5 @@
 <robot xmlns:xacro="http://www.ros.org/wiki/xacro" name="revo2_left">
     <xacro:arg name="initial_positions_file" default="revo2_left_initial_positions.yaml" />
-    <xacro:arg name="ctrl_param_duration_ms" default="10" />
+    <xacro:arg name="ctrl_param_duration_ms" default="55" />
     <!-- World link -->
     <link name="world"/>

File: brainco_hardware/stark_ethercat/brainco_hand_ethercat_driver/config/revo2_right.ros2_control.xacro (robot description, xacro)
@@ -1,5 +1,5 @@
 <?xml version="1.0"?>
 <robot xmlns:xacro="http://www.ros.org/wiki/xacro">
-    <xacro:macro name="revo2_right_ros2_control" params="name initial_positions_file ctrl_param_duration_ms:=10">
+    <xacro:macro name="revo2_right_ros2_control" params="name initial_positions_file ctrl_param_duration_ms:=55">
         <xacro:property name="initial_positions" value="${xacro.load_yaml(initial_positions_file)['initial_positions']}"/>
         <ros2_control name="${name}" type="system">

File: brainco_hardware/stark_ethercat/brainco_hand_ethercat_driver/config/revo2_right.urdf.xacro (robot description, xacro)
@@ -2,5 +2,5 @@
 <robot xmlns:xacro="http://www.ros.org/wiki/xacro" name="revo2_right">
     <xacro:arg name="initial_positions_file" default="revo2_right_initial_positions.yaml" />
-    <xacro:arg name="ctrl_param_duration_ms" default="10" />
+    <xacro:arg name="ctrl_param_duration_ms" default="55" />
     <!-- World link -->
     <link name="world"/>
